File: hw/bank34_35.kicad_sch (KiCad schematic)
At the start: 15 parts, among them U24 XC7A35T-FTG256

Commit message: WIP (layout)
Parts:
- removed C50: 470n, Capacitor_SMD:C_0402_1005Metric, symbol Device:C_Small
- removed C51: 4u7, Capacitor_SMD:C_0805_2012Metric, symbol Device:C_Small
Changed lines of the file:
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@@
   (junction (at 109.22 21.59) (diameter 0) (color 0 0 0 0)
   )
-  (junction (at 99.06 26.67) (diameter 0) (color 0 0 0 0)
-  )
   (junction (at 119.38 21.59) (diameter 0) (color 0 0 0 0)
   )
   (junction (at 137.16 35.56) (diameter 0) (color 0 0 0 0)
   )
-  (junction (at 99.06 21.59) (diameter 0) (color 0 0 0 0)
-  )
   (junction (at 76.2 26.67) (diameter 0) (color 0 0 0 0)
   )
@@
   (junction (at 139.7 35.56) (diameter 0) (color 0 0 0 0)
   )
-  (junction (at 86.36 26.67) (diameter 0) (color 0 0 0 0)
-  )
   (junction (at 160.02 30.48) (diameter 0) (color 0 0 0 0)
   )
@@
   (junction (at 76.2 21.59) (diameter 0) (color 0 0 0 0)
   )
-  (junction (at 86.36 21.59) (diameter 0) (color 0 0 0 0)
-  )
   (junction (at 132.08 35.56) (diameter 0) (color 0 0 0 0)
   )
@@
     (stroke (width 0) (type default))
   )
-  (wire (pts (xy 86.36 26.67) (xy 76.2 26.67))
-    (stroke (width 0) (type default))
-  )
   (wire (pts (xy 58.42 31.75) (xy 58.42 35.56))
     (stroke (width 0) (type default))
@@
     (stroke (width 0) (type default))
   )
-  (wire (pts (xy 99.06 26.67) (xy 109.22 26.67))
+  (wire (pts (xy 76.2 26.67) (xy 109.22 26.67))
     (stroke (width 0) (type default))
   )
@@
     (stroke (width 0) (type default))
   )
-  (wire (pts (xy 86.36 21.59) (xy 76.2 21.59))
+  (wire (pts (xy 76.2 21.59) (xy 109.22 21.59))
     (stroke (width 0) (type default))
   )
@@
     (stroke (width 0) (type default))
   )
-  (wire (pts (xy 86.36 21.59) (xy 99.06 21.59))
-    (stroke (width 0) (type default))
-  )
   (wire (pts (xy 182.88 30.48) (xy 193.04 30.48))
     (stroke (width 0) (type default))
@@
     (stroke (width 0) (type default))
   )
-  (wire (pts (xy 86.36 26.67) (xy 99.06 26.67))
-    (stroke (width 0) (type default))
-  )
   (wire (pts (xy 109.22 21.59) (xy 119.38 21.59))
     (stroke (width 0) (type default))
@@
   )
   (wire (pts (xy 63.5 31.75) (xy 63.5 35.56))
-    (stroke (width 0) (type default))
-  )
-  (wire (pts (xy 99.06 21.59) (xy 109.22 21.59))
     (stroke (width 0) (type default))
   )
@@
         (path "/ad7ba5e2-7ca2-4db6-ac22-68607f85c2e2"
           (reference "C53") (unit 1)
-        )
-      )
-    )
-  )
-  (symbol (lib_id "Device:C_Small") (at 99.06 24.13 0) (unit 1)
-    (in_bom yes) (on_board yes) (dnp no)
-    (property "Reference" "C50" (at 101.3968 22.9616 0)
-      (effects (font (size 1.27 1.27)) (justify left))
-    )
-    (property "Value" "470n" (at 101.3968 25.273 0)
-      (effects (font (size 1.27 1.27)) (justify left))
-    )
-    (property "Footprint" "Capacitor_SMD:C_0402_1005Metric" (at 99.06 24.13 0)
-      (effects (font (size 1.27 1.27)) hide)
-    )
-    (property "Datasheet" "~" (at 99.06 24.13 0)
-      (effects (font (size 1.27 1.27)) hide)
-    )
-    (pin "1")
-    (pin "2")
-    (instances
-      (project "ecevr-proto"
-        (path "/0333b818-5fb1-4de6-9929-c91b1fef8666/00000000-0000-0000-0000-0000620d1e32/00000000-0000-0000-0000-00006209ff9a"
-          (reference "C50") (unit 1)
-        )
-      )
-      (project "usbadc"
-        (path "/7c8a1f8d-8834-4c9b-aaae-1f231e9b09a1/27cc8612-21b5-4a6c-80ae-cd0836a5c2c4/3e711749-c38a-4641-a750-86491e73d656"
-          (reference "C158") (unit 1)
-        )
-      )
-      (project "bank34_35"
-        (path "/ad7ba5e2-7ca2-4db6-ac22-68607f85c2e2"
-          (reference "C50") (unit 1)
         )
       )
@@
         )
       )
-    )
-  )
-  (symbol (lib_id "Device:C_Small") (at 86.36 24.13 0) (unit 1)
-    (in_bom yes) (on_board yes) (dnp no)
-    (property "Reference" "C51" (at 88.6968 22.9616 0)
-      (effects (font (size 1.27 1.27)) (justify left))
-    )
-    (property "Value" "4u7" (at 88.6968 25.273 0)
-      (effects (font (size 1.27 1.27)) (justify left))
-    )
-    (property "Footprint" "Capacitor_SMD:C_0805_2012Metric" (at 86.36 24.13 0)
-      (effects (font (size 1.27 1.27)) hide)
-    )
-    (property "Datasheet" "~" (at 86.36 24.13 0)
-      (effects (font (size 1.27 1.27)) hide)
-    )
-    (pin "1")
-    (pin "2")
-    (instances
-      (project "ecevr-proto"
-        (path "/0333b818-5fb1-4de6-9929-c91b1fef8666/00000000-0000-0000-0000-0000620d1e32/00000000-0000-0000-0000-00006209ff9a"
-          (reference "C51") (unit 1)
-        )
-      )
-      (project "usbadc"
-        (path "/7c8a1f8d-8834-4c9b-aaae-1f231e9b09a1/27cc8612-21b5-4a6c-80ae-cd0836a5c2c4/3e711749-c38a-4641-a750-86491e73d656"
-          (reference "C157") (unit 1)
-        )
-      )
-      (project "bank34_35"
-        (path "/ad7ba5e2-7ca2-4db6-ac22-68607f85c2e2"
-          (reference "C51") (unit 1)
-        )
-      )
