File: hw/bank_0.kicad_sch (KiCad schematic)
At the start: 8 parts, among them SW1 PROG, U24 XC7A35T-FTG256

Commit message: layout finished (draft)
Parts:
- JP1, JP2: symbol Device:Jumper_NO_Small -> Jumper:Jumper_2_Open
Changed lines of the file:
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@@
   (junction (at 111.76 134.62) (diameter 0) (color 0 0 0 0)
   )
-  (junction (at 114.3 101.6) (diameter 0) (color 0 0 0 0)
-  )
   (junction (at 111.76 129.54) (diameter 0) (color 0 0 0 0)
   )
@@
   (junction (at 161.29 114.3) (diameter 0) (color 0 0 0 0)
   )
-  (junction (at 151.13 128.27) (diameter 0) (color 0 0 0 0)
+  (junction (at 149.86 128.27) (diameter 0) (color 0 0 0 0)
   )
   (junction (at 140.97 116.84) (diameter 0) (color 0 0 0 0)
@@
     (stroke (width 0) (type default))
   )
-  (wire (pts (xy 134.62 109.22) (xy 134.62 107.95))
-    (stroke (width 0) (type default))
-  )
   (wire (pts (xy 130.81 121.92) (xy 125.73 121.92))
     (stroke (width 0) (type default))
@@
     (stroke (width 0) (type default))
   )
-  (wire (pts (xy 151.13 128.27) (xy 151.13 121.92))
-    (stroke (width 0) (type default))
-  )
-  (wire (pts (xy 151.13 121.92) (xy 154.94 121.92))
+  (wire (pts (xy 149.86 128.27) (xy 149.86 121.92))
     (stroke (width 0) (type default))
   )
@@
     (stroke (width 0) (type default))
   )
-  (wire (pts (xy 134.62 101.6) (xy 114.3 101.6))
-    (stroke (width 0) (type default))
-  )
   (wire (pts (xy 111.76 132.08) (xy 111.76 134.62))
     (stroke (width 0) (type default))
@@
     (stroke (width 0) (type default))
   )
-  (wire (pts (xy 114.3 109.22) (xy 134.62 109.22))
+  (wire (pts (xy 146.05 97.79) (xy 153.67 97.79))
     (stroke (width 0) (type default))
   )
@@
     (stroke (width 0) (type default))
   )
-  (wire (pts (xy 134.62 102.87) (xy 134.62 101.6))
-    (stroke (width 0) (type default))
-  )
   (wire (pts (xy 116.84 86.36) (xy 111.76 86.36))
     (stroke (width 0) (type default))
@@
     (stroke (width 0) (type default))
   )
-  (wire (pts (xy 135.89 128.27) (xy 151.13 128.27))
+  (wire (pts (xy 135.89 128.27) (xy 149.86 128.27))
+    (stroke (width 0) (type default))
+  )
+  (wire (pts (xy 146.05 98.425) (xy 146.05 97.79))
     (stroke (width 0) (type default))
   )
@@
   )
   (wire (pts (xy 111.76 106.68) (xy 114.3 106.68))
+    (stroke (width 0) (type default))
+  )
+  (wire (pts (xy 114.3 109.22) (xy 146.05 109.22))
+    (stroke (width 0) (type default))
+  )
+  (wire (pts (xy 146.05 109.22) (xy 146.05 108.585))
     (stroke (width 0) (type default))
   )
@@
     (effects (font (size 1.27 1.27)) (justify left))
   )
-  (symbol (lib_id "Device:Jumper_NO_Small") (at 157.48 121.92 180) (unit 1)
-    (in_bom yes) (on_board yes) (dnp no)
-    (property "Reference" "JP2" (at 156.21 125.73 90)
-      (effects (font (size 1.27 1.27)))
-    )
-    (property "Value" "INITb" (at 158.75 125.73 90)
-      (effects (font (size 1.27 1.27)))
-    )
-    (property "Footprint" "Connector_PinHeader_2.54mm:PinHeader_1x02_P2.54mm_Vertical" (at 157.48 121.92 0)
-      (effects (font (size 1.27 1.27)) hide)
-    )
-    (property "Datasheet" "~" (at 157.48 121.92 0)
+  (symbol (lib_id "Jumper:Jumper_2_Open") (at 154.94 121.92 180) (unit 1)
+    (in_bom yes) (on_board yes) (dnp no)
+    (property "Reference" "JP2" (at 153.67 125.73 90)
+      (effects (font (size 1.27 1.27)))
+    )
+    (property "Value" "INITb" (at 156.21 125.73 90)
+      (effects (font (size 1.27 1.27)))
+    )
+    (property "Footprint" "Connector_PinHeader_2.54mm:PinHeader_1x02_P2.54mm_Vertical" (at 154.94 121.92 0)
+      (effects (font (size 1.27 1.27)) hide)
+    )
+    (property "Datasheet" "~" (at 154.94 121.92 0)
       (effects (font (size 1.27 1.27)) hide)
     )
@@
     )
   )
-  (symbol (lib_id "Device:Jumper_NO_Small") (at 134.62 105.41 270) (unit 1)
-    (in_bom yes) (on_board yes) (dnp no)
-    (property "Reference" "JP1" (at 138.43 106.68 90)
-      (effects (font (size 1.27 1.27)))
-    )
-    (property "Value" "JTAG_boot" (at 140.97 104.14 90)
-      (effects (font (size 1.27 1.27)))
-    )
-    (property "Footprint" "Connector_PinHeader_2.54mm:PinHeader_1x02_P2.54mm_Vertical" (at 134.62 105.41 0)
-      (effects (font (size 1.27 1.27)) hide)
-    )
-    (property "Datasheet" "~" (at 134.62 105.41 0)
+  (symbol (lib_id "Jumper:Jumper_2_Open") (at 146.05 103.505 90) (mirror x) (unit 1)
+    (in_bom yes) (on_board yes) (dnp no)
+    (property "Reference" "JP1" (at 142.24 104.775 90)
+      (effects (font (size 1.27 1.27)))
+    )
+    (property "Value" "JTAG_boot" (at 139.7 102.235 90)
+      (effects (font (size 1.27 1.27)))
+    )
+    (property "Footprint" "Connector_PinHeader_2.54mm:PinHeader_1x02_P2.54mm_Vertical" (at 146.05 103.505 0)
+      (effects (font (size 1.27 1.27)) hide)
+    )
+    (property "Datasheet" "~" (at 146.05 103.505 0)
       (effects (font (size 1.27 1.27)) hide)
     )
@@
     )
   )
-  (symbol (lib_id "power:GND") (at 151.13 128.27 0) (unit 1)
-    (in_bom yes) (on_board yes) (dnp no)
-    (property "Reference" "#PWR0141" (at 151.13 134.62 0)
-      (effects (font (size 1.27 1.27)) hide)
-    )
-    (property "Value" "GND" (at 151.257 132.6642 0)
-      (effects (font (size 1.27 1.27)))
-    )
-    (property "Footprint" "" (at 151.13 128.27 0)
-      (effects (font (size 1.27 1.27)) hide)
-    )
-    (property "Datasheet" "" (at 151.13 128.27 0)
-      (effects (font (size 1.27 1.27)) hide)
-    )
+  (symbol (lib_id "power:GND") (at 149.86 128.27 0) (unit 1)
+    (in_bom yes) (on_board yes) (dnp no)
+    (property "Reference" "#PWR0141" (at 149.86 134.62 0)
+      (effects (font (size 1.27 1.27)) hide)
+    )
+    (property "Value" "GND" (at 149.987 132.6642 0)
+      (effects (font (size 1.27 1.27)))
+    )
+    (property "Footprint" "" (at 149.86 128.27 0)
+      (effects (font (size 1.27 1.27)) hide)
+    )
+    (property "Datasheet" "" (at 149.86 128.27 0)
+      (effects (font (size 1.27 1.27)) hide)
+    )
