File: hw/usbadc.kicad_pcb (KiCad board)
At the start: 4 copper layers, 100 x 60 mm, 332 parts, among them J1 USB_C_Receptacle_USB2.0, J2 BNC, J3 BNC, J4 T8_JTAG, J5 BNC, J7 BNC, J9 Expansion, K1 G6S-2, K2 G6S-2, Q1 SSM6N35AFE, Q10 SSM6N35AFE, Q12 SSM6N35AFE, Q13 SSM6N35AFE, Q2 SSM6N35AFE, Q3 SSM6N35AFE, Q4 SSM6P35AFE, Q5 SSM6P35AFE, Q6 SSM6N35AFE, Q7 SSM6N35AFE, Q8 DMC2053UVT, Q9 SSM6N35AFE, SW1 Reconfig, U1 RT8096B, U10 AQY225R2S, U11 TS5A63157DBV, U12 OPA859xDSG, U13 AD8370, U14 AQY225R2S, U15 T20Q144xx, U16 USB3343, U17 NDS36PT5-16ET, U18 TS5A63157DBV, U19 OPA859xDSG, U2 RT8096B, U20 AD8370, U22 TSV992A, U23 MCP47CVB02-E_UN, U24 AT25FF081A-SSHN-B, U3 RT8096B, U4 SN74LVC2T45DCUR, U5 TPS563249DDC, U6 PCA9306, U7 5P49V5925, U8 24AA0x, U9 MAX19517, X1 ECS-2520MV-260-CN-TR, Y1 26MHz

Commit message: updated some component values
Parts:
- C14: value 50p -> 47p
- FB2: value Ferrite_Bead -> Ferrite_Bead MPZ1608S221A
- R70: value 5k1 -> 2k2
- U6: value PCA9306 -> PCA9306DC1
- Y1: value 26MHz -> 25MHz
Changed lines of the file:
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@@
         (effects (font (size 1 1) (thickness 0.15)))
     )
-    (fp_text value "50p" (at 0 1.43) (layer "F.Fab")
+    (fp_text value "47p" (at 0 1.43) (layer "F.Fab")
         (effects (font (size 1 1) (thickness 0.15)))
     )
@@
         (effects (font (size 1 1) (thickness 0.15)))
     )
-    (fp_text value "5k1" (at 0 1.43) (layer "F.Fab")
+    (fp_text value "2k2" (at 0 1.43) (layer "F.Fab")
         (effects (font (size 1 1) (thickness 0.15)))
     )
@@
         (effects (font (size 1 1) (thickness 0.15)))
     )
-    (fp_text value "PCA9306" (at 0 2.413) (layer "F.Fab")
+    (fp_text value "PCA9306DC1" (at 0 2.413) (layer "F.Fab")
         (effects (font (size 1 1) (thickness 0.15)))
     )
@@
         (effects (font (size 1 1) (thickness 0.15)))
     )
-    (fp_text value "Ferrite_Bead" (at 0 1.43) (layer "F.Fab")
+    (fp_text value "Ferrite_Bead MPZ1608S221A" (at 0 1.43) (layer "F.Fab")
         (effects (font (size 1 1) (thickness 0.15)))
     )
@@
     (tags "SMD SMT crystal Abracon ABM10")
     (property "Manufacturer" "Abracon")
-    (property "Part" "ABM10W-26.0000MHZ-8-B1U-T3")
+    (property "Part" "ABM10W-25.0000MHZ-8-B1U-T3")
     (property "Sheetfile" "pll_clock.kicad_sch")
     (property "Sheetname" "Clock")
@@
         (effects (font (size 1 1) (thickness 0.15)))
     )
-    (fp_text value "26MHz" (at 0.04 2.5 90) (layer "F.Fab")
+    (fp_text value "25MHz" (at 0.04 2.5 90) (layer "F.Fab")
         (effects (font (size 1 1) (thickness 0.15)))
     )

Commit message: PGA_SDAT / PGA_LATCH_CHB were swapped in top-sheet
 -> corrected there and swapped at FPGA bank keeps the
 layout unmodified but fixes the labels.
 => still compatible with v3.0 as ordered from JLC
Connections:
- Q5 pad 2: PGA_LATCH_CHB -> PGA_SDAT
- Q5 pad 5: PGA_SDAT -> PGA_LATCH_CHB
- U15 pad 65: PGA_LATCH_CHB -> PGA_SDAT
- U15 pad 67: PGA_SDAT -> PGA_LATCH_CHB
Routing:
- net PGA_SDAT: track 20.0 -> 20.8 mm
- net PGA_LATCH_CHB: track 20.8 -> 20.0 mm
Changed lines of the file:
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@@
       (net 1 "GND") (pinfunction "GND") (pintype "passive"))
     (pad "65" smd roundrect (at 5.25 10.6625) (size 0.3 1.475) (layers "F.Cu" "F.Paste" "F.Mask") (roundrect_rratio 0.25)
-      (net 271 "PGA_LATCH_CHB") (pinfunction "GPIOB_RXN07") (pintype "bidirectional"))
+      (net 270 "PGA_SDAT") (pinfunction "GPIOB_RXN07") (pintype "bidirectional"))
     (pad "66" smd roundrect (at 5.75 10.6625) (size 0.3 1.475) (layers "F.Cu" "F.Paste" "F.Mask") (roundrect_rratio 0.25)
       (net 32 "ADC_SYNC") (pinfunction "GPIOB_RXP07") (pintype "bidirectional"))
     (pad "67" smd roundrect (at 6.25 10.6625) (size 0.3 1.475) (layers "F.Cu" "F.Paste" "F.Mask") (roundrect_rratio 0.25)
-      (net 270 "PGA_SDAT") (pinfunction "GPIOB_RXP10") (pintype "bidirectional"))
+      (net 271 "PGA_LATCH_CHB") (pinfunction "GPIOB_RXP10") (pintype "bidirectional"))
     (pad "68" smd roundrect (at 6.75 10.6625) (size 0.3 1.475) (layers "F.Cu" "F.Paste" "F.Mask") (roundrect_rratio 0.25)
       (net 268 "PGA_LATCH_CHA") (pinfunction "GPIOB_RXN10") (pintype "bidirectional"))
@@
       (net 96 "+2V5_analog") (pinfunction "S") (pintype "passive"))
     (pad "2" smd rect (at -0.635 0 90) (size 0.67 0.3) (layers "F.Cu" "F.Paste" "F.Mask")
-      (net 271 "PGA_LATCH_CHB") (pinfunction "G") (pintype "input"))
+      (net 270 "PGA_SDAT") (pinfunction "G") (pintype "input"))
     (pad "3" smd rect (at -0.635 0.5 90) (size 0.67 0.3) (layers "F.Cu" "F.Paste" "F.Mask")
       (net 52 "/Front End/FE_CHB/PGA_CTL_LATCH") (pinfunction "D") (pintype "passive"))
@@
       (net 96 "+2V5_analog") (pinfunction "S") (pintype "passive"))
     (pad "5" smd rect (at 0.635 0 90) (size 0.67 0.3) (layers "F.Cu" "F.Paste" "F.Mask")
-      (net 270 "PGA_SDAT") (pinfunction "G") (pintype "input"))
+      (net 271 "PGA_LATCH_CHB") (pinfunction "G") (pintype "input"))
     (pad "6" smd rect (at 0.635 -0.5 90) (size 0.67 0.3) (layers "F.Cu" "F.Paste" "F.Mask")
       (net 49 "/Front End/FE_CHA/PGA_CTL_DATA") (pinfunction "D") (pintype "passive"))
@@
   (segment (start 119.2 72.175) (end 119.2 72.56) (width 0.1) (layer "F.Cu") (net 269))
   (segment (start 118.875 71.85) (end 119.2 72.175) (width 0.1) (layer "F.Cu") (net 269))
-  (segment (start 117.875 75.325) (end 119 75.325) (width 0.1) (layer "F.Cu") (net 270))
-  (segment (start 114.525 77.1) (end 116.1 77.1) (width 0.1) (layer "F.Cu") (net 270))
-  (segment (start 119.2 75.125) (end 119.2 74.83) (width 0.1) (layer "F.Cu") (net 270))
-  (segment (start 106.4 80.025) (end 111.6 80.025) (width 0.1) (layer "F.Cu") (net 270))
-  (segment (start 103.5985 77.2235) (end 106.4 80.025) (width 0.1) (layer "F.Cu") (net 270))
-  (segment (start 116.1 77.1) (end 117.875 75.325) (width 0.1) (layer "F.Cu") (net 270))
-  (segment (start 111.6 80.025) (end 114.525 77.1) (width 0.1) (layer "F.Cu") (net 270))
-  (segment (start 103.5985 76.3415) (end 103.5985 77.2235) (width 0.1) (layer "F.Cu") (net 270))
-  (segment (start 119 75.325) (end 119.2 75.125) (width 0.1) (layer "F.Cu") (net 270))
-  (segment (start 119.2 75.875) (end 119.2 76.1) (width 0.1) (layer "F.Cu") (net 271))
-  (segment (start 105.9 80.225) (end 111.682842 80.225) (width 0.1) (layer "F.Cu") (net 271))
-  (segment (start 102.5985 76.3415) (end 102.5985 76.9235) (width 0.1) (layer "F.Cu") (net 271))
-  (segment (start 114.607842 77.3) (end 116.275 77.3) (width 0.1) (layer "F.Cu") (net 271))
-  (segment (start 116.275 77.3) (end 118 75.575) (width 0.1) (layer "F.Cu") (net 271))
-  (segment (start 118 75.575) (end 118.9 75.575) (width 0.1) (layer "F.Cu") (net 271))
-  (segment (start 102.5985 76.9235) (end 105.9 80.225) (width 0.1) (layer "F.Cu") (net 271))
-  (segment (start 118.9 75.575) (end 119.2 75.875) (width 0.1) (layer "F.Cu") (net 271))
-  (segment (start 111.682842 80.225) (end 114.607842 77.3) (width 0.1) (layer "F.Cu") (net 271))
+  (segment (start 119.2 75.875) (end 119.2 76.1) (width 0.1) (layer "F.Cu") (net 270))
+  (segment (start 105.9 80.225) (end 111.682842 80.225) (width 0.1) (layer "F.Cu") (net 270))
+  (segment (start 102.5985 76.3415) (end 102.5985 76.9235) (width 0.1) (layer "F.Cu") (net 270))
+  (segment (start 114.607842 77.3) (end 116.275 77.3) (width 0.1) (layer "F.Cu") (net 270))
+  (segment (start 116.275 77.3) (end 118 75.575) (width 0.1) (layer "F.Cu") (net 270))
+  (segment (start 118 75.575) (end 118.9 75.575) (width 0.1) (layer "F.Cu") (net 270))
+  (segment (start 102.5985 76.9235) (end 105.9 80.225) (width 0.1) (layer "F.Cu") (net 270))
+  (segment (start 118.9 75.575) (end 119.2 75.875) (width 0.1) (layer "F.Cu") (net 270))
+  (segment (start 111.682842 80.225) (end 114.607842 77.3) (width 0.1) (layer "F.Cu") (net 270))
+  (segment (start 117.875 75.325) (end 119 75.325) (width 0.1) (layer "F.Cu") (net 271))
+  (segment (start 114.525 77.1) (end 116.1 77.1) (width 0.1) (layer "F.Cu") (net 271))
+  (segment (start 119.2 75.125) (end 119.2 74.83) (width 0.1) (layer "F.Cu") (net 271))
+  (segment (start 106.4 80.025) (end 111.6 80.025) (width 0.1) (layer "F.Cu") (net 271))
+  (segment (start 103.5985 77.2235) (end 106.4 80.025) (width 0.1) (layer "F.Cu") (net 271))
+  (segment (start 116.1 77.1) (end 117.875 75.325) (width 0.1) (layer "F.Cu") (net 271))
+  (segment (start 111.6 80.025) (end 114.525 77.1) (width 0.1) (layer "F.Cu") (net 271))
+  (segment (start 103.5985 76.3415) (end 103.5985 77.2235) (width 0.1) (layer "F.Cu") (net 271))
+  (segment (start 119 75.325) (end 119.2 75.125) (width 0.1) (layer "F.Cu") (net 271))
   (segment (start 90.0985 76.3415) (end 90.0985 77.381) (width 0.1) (layer "F.Cu") (net 272))
   (segment (start 90.0985 77.381) (end 90.0945 77.385) (width 0.1) (layer "F.Cu") (net 272))
