File: hw/fe_ctl.kicad_sch (KiCad schematic)
At the start: 3 parts, among them U21 TCA6408A

Commit message: renaming, comments, part/vendor and other cosmetics (no pcb change)
Parts:
- U21: Manufacturer (none) -> TI; Part (none) -> TCA6408ARGTR
Changed lines of the file:
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@@
+      (effects (font (size 1.27 1.27)) hide)
+    )
+    (property "Part" "TCA6408ARGTR" (at 124.46 99.06 0)
+      (effects (font (size 1.27 1.27)) hide)
+    )
+    (property "Manufacturer" "TI" (at 124.46 99.06 0)
       (effects (font (size 1.27 1.27)) hide)
     )

Commit message: WIP: intermediate commit (routing)
will try to update library footprints
Parts:
- added C9: 100n, Capacitor_SMD:C_0603_1608Metric, symbol Device:C_Small
Connections:
- net +4V: now also C9.1
- net GND: now also C9.2
Other:
- moved on the sheet: C140

Commit message: updated parts assignments
Parts:
- R60: Manufacturer (none) -> Stackpole; Part (none) -> RMCF0603FT10K0
Changed lines of the file:
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@@
 			)
 		)
-		(property "Part" ""
+		(property "Part" "RMCF0603FT10K0"
 			(at 111.76 88.9 90)
 			(effects
@@
 			)
 		)
-		(property "Manufacturer" ""
+		(property "Manufacturer" "Stackpole"
 			(at 111.76 88.9 90)
 			(effects

Commit message: connected versaclock CLKSEL to ULPI RSTB (share FPGA pin)
ULPI Rstb is unlikely to be used

Also: - update of kicad to 9.0 (many library footprints updated)
      - added sheet titles, author
Other:
- company: (none) -> Till Straumann
- title: (none) -> IO Extender / Level Shifter

Commit message: Added licensing information
Other:
- company: Till Straumann -> Copyright Till Straumann, 2025
Changed lines of the file:
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@@
 		(title "IO Extender / Level Shifter")
 		(rev "3.3b")
-		(company "Till Straumann")
-		(comment 1 "4V I/O Voltage for relays and analog switches")
+		(company "Copyright Till Straumann, 2025")
+		(comment 1 "License: CERN-OHL-P v2")
 	)
 	(text "NOTES:\nI2C Address 0x40\nADDR: VCCp levels\nRESETb: VCCi levels\nPAD: seems unconnected"
