File: hw/leds.kicad_sch (KiCad schematic)
At the start: 22 parts, among them Q2 SSM3K37MFV

Commit message: Added licensing information
Other:
- company: Till Straumann -> Copyright Till Straumann, 2025
Changed lines of the file:
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@@
 		(title "LEDs")
 		(rev "3.3b")
-		(company "Till Straumann")
+		(company "Copyright Till Straumann, 2025")
+		(comment 1 "License: CERN-OHL-P v2")
 	)
 	(text "RED"
