File: hw/buffer.kicad_sch (KiCad schematic)
At the start: 40 parts, among them J1001 BNC, J1002 RFShield_Front, J1003 RFShield_Back, J2 RFShield_Back_Cover, J6 RFShield_Back_Front, K1001 G6L-1F, U1001 TS5A63157DCK, U1002 AQY280S, U1003 AD8370, U1004 OPA859xDSG

Commit message: added some comments in schematics
Other:
- note added: "Analog switch controls 0db/-20db switchable buffer/attenuator"
- note added: "Mechanical relay controls 50-ohm termination"
- note added: "Solid-state relay controls AC/DC coupling"
Changed lines of the file:
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@@
 		(comment 1 "License: CERN-OHL-P v2")
+	)
+	(text "Analog switch controls\n0db/-20db switchable\nbuffer/attenuator"
+		(exclude_from_sim no)
+		(at 125.73 36.83 0)
+		(effects
+			(font
+				(size 1.27 1.27)
+			)
+			(justify left)
+		)
+	)
+	(text "Mechanical relay\ncontrols 50-ohm\ntermination"
+		(exclude_from_sim no)
+		(at 81.28 36.83 0)
+		(effects
+			(font
+				(size 1.27 1.27)
+			)
+			(justify left)
+		)
 	)
 	(text "Ideally: 101k//99p but\n99p is not available"
@@
 		)
 	)
+	(text "Solid-state relay\ncontrols AC/DC\ncoupling"
+		(exclude_from_sim no)
+		(at 53.34 36.83 0)
+		(effects
+			(font
+				(size 1.27 1.27)
+			)
+			(justify left)
+		)
+	)
