File: hw/front_end.kicad_sch (KiCad schematic)
At the start: 11 parts, among them Q4 SSM6P35AFE, Q5 SSM6P35AFE, Q6 SSM6P35AFE

Commit message: added some comments in schematics
Other:
- note added: "Level shifters for PGA serial interface"
Changed lines of the file:
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@@
+		)
+	)
+	(text "Level shifters for PGA\nserial interface"
+		(exclude_from_sim no)
+		(at 29.21 44.45 0)
+		(effects
+			(font
+				(size 1.27 1.27)
+			)
+			(justify left)
 		)
 	)
