File: hw/max19507.kicad_sch (KiCad schematic)
At the start: 31 parts, among them U9 MAX19517

Commit message: added some comments in schematics
Other:
- note added: "Input protection diodes"
Changed lines of the file:
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@@
+		)
+	)
+	(text "Input protection diodes"
+		(exclude_from_sim no)
+		(at 130.81 156.21 0)
+		(effects
+			(font
+				(size 1.27 1.27)
+			)
 		)
 	)
