File: hw/sdram.kicad_sch (KiCad schematic)
At the start: 25 parts, among them U15 T20Q144xx, U17 NDS36PT5-16ET

Commit message: added some comments in schematics
Other:
- note added: "Prevent ADC from driving ADC_D7..D9 by pulling up ADC_SHDN. Ensures the CBUS configuration pins are pulled up. Once configured the FPGA can drive ADC_SHDN low to activate the ADC."
- note removed: "Prevent ADC from driving ADC_D7..D9 by pulling up ADC_SHDN. Ensures the CBUS configuration pins are pulled up. Once configured the FPGA can drive ADC_SHDN low to activate."
Changed lines of the file:
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@@
 		(comment 1 "License: CERN-OHL-P v2")
 	)
-	(text "Prevent ADC from driving ADC_D7..D9\nby pulling up ADC_SHDN. Ensures the\nCBUS configuration pins are pulled\nup. Once configured the FPGA can drive\nADC_SHDN low to activate."
+	(text "Prevent ADC from driving ADC_D7..D9\nby pulling up ADC_SHDN. Ensures the\nCBUS configuration pins are pulled\nup. Once configured the FPGA can drive\nADC_SHDN low to activate the ADC."
 		(exclude_from_sim no)
 		(at 40.005 147.955 0)
